File: schema/atmega-z80.kicad_pcb (KiCad board)
At the start: 2 copper layers, 142.2 x 115.6 mm, 75 parts, among them J1 USB Connector, J2 Programmer ISP 10, J3 SPI Connector, J4 I2C Connector, Q1 PNP_2N4403, Q2 PNP_2N4403, Q3 NPN_2N4401, Q4 PNP_2N4403, U1 Z84C0010PEG, U2 ATmega324A-PU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

Commit message: Changed #Z80_RESET line pull-down (R13) to pull-up
Parts:
- moved R13 45.3 mm to (117.9, 87.3), turned to 270 degrees
Connections:
- R13 pad 1: GND -> +5V
Routing:
- net /#RD: track 69.1 -> 152.5 mm, vias 0 -> 2
- net /#WR: track 0.00 -> 78.6 mm, vias 0 -> 2
- net /#INT: track 0.00 -> 41.5 mm, vias 0 -> 3
- net /#Z80_RESET: track 3.56 -> 30.2 mm, vias 0 -> 1
- net +5V: track 662.4 -> 665.1 mm
- net /#Z80_CLK: track 66.8 -> 69.3 mm
- net /D3: track 155.6 -> 156.7 mm
- net #MEM_LED: track 203.2 -> 202.2 mm
- net GND: vias 146 -> 154
